File: mxm immobilizer/mxm_immobilizer.kicad_sch (KiCad schematic)
At the start: 381 parts, among them J1 PEX_STD_SW#_SWITCH, J10 LVDS_VOLTAGE_SWITCH, J11 LVDS_header_30p, J2 VGA_DISABLE#_SWITCH, J3 3V3_SWITCH, J4 PWR_LEVEL_SWITCH, J5 PWR_EN_SWITCH, J6 TH_ALERT#_SWITCH, J7 Clevo_MXM_PWR, J8 MXM_JTAG, J9 5V_SWITCH, M1 Fan_Tacho_PWM, Q1 2N7002, Q10 2N7002, Q11 2N7002, Q12 2N7002, Q13 2N7002, Q14 2N7002, Q15 2N7002, Q16 2N7002, Q17 2N7002, Q18 2N7002, Q19 2N7002, Q2 2N7002, Q20 2N7002, Q21 2N7002, Q22 2N7002, Q23 2N7002, Q24 2N7002, Q25 2N7002, Q26 2N7002, Q27 2N7002, Q28 2N7002, Q29 2N7002, Q3 2N7002, Q30 2N7002, Q31 2N7002, Q32 2N7002, Q33 2N7002, Q34 2N7002, Q35 2N7002, Q36 2N7002, Q4 2N7002, Q5 2N7002, Q6 2N7002, Q7 2N7002, Q8 2N7002, Q9 2N7002, SW1 TH_OVERT#_RESET, U1 sy6280, U2 sy6280, U3 74LVC1G373, U4 LM2596S-5

Commit message: Added PCIe Rx capacitors (and updated to KiCad 9)
should've done this ages ago...
Parts:
- added C117, C118, C119, C120, C121, C122, C123, C124, C125, C126, C127, C128, C129, C130, C131, C132, C133, C134, C135, C136, C137, C138, C139, C140, C141, C142, C143, C144, C145, C146, C147, C148: 0.22uF, Capacitor_SMD:C_0402_1005Metric, symbol Device:C_Small
Connections:
- net RX0+: now also C118.1; no longer MXM1.147 (PEX_RX0#)
- net RX0-: now also C117.1; no longer MXM1.149 (PEX_RX0)
- net RX1+: now also C120.1; no longer MXM1.141 (PEX_RX1#)
- net RX1-: now also C119.1; no longer MXM1.143 (PEX_RX1)
- net RX10+: now also C138.1; no longer MXM1.79 (PEX_RX10#)
- net RX10-: now also C137.1; no longer MXM1.81 (PEX_RX10)
- net RX11+: now also C140.1; no longer MXM1.73 (PEX_RX11#)
- net RX11-: now also C139.1; no longer MXM1.75 (PEX_RX11)
- net RX12+: now also C142.1; no longer MXM1.67 (PEX_RX12#)
- net RX12-: now also C141.1; no longer MXM1.69 (PEX_RX12)
- net RX13+: now also C144.1; no longer MXM1.61 (PEX_RX13#)
- net RX13-: now also C143.1; no longer MXM1.63 (PEX_RX13)
- net RX14+: now also C146.1; no longer MXM1.55 (PEX_RX14#)
- net RX14-: now also C145.1; no longer MXM1.57 (PEX_RX14)
- net RX15+: now also C148.1; no longer MXM1.49 (PEX_RX15#)
- net RX15-: now also C147.1; no longer MXM1.51 (PEX_RX15)
- net RX2+: now also C122.1; no longer MXM1.135 (PEX_RX2#)
- net RX2-: now also C121.1; no longer MXM1.137 (PEX_RX2)
- net RX3+: now also C124.1; no longer MXM1.121 (PEX_RX3#)
- net RX3-: now also C123.1; no longer MXM1.123 (PEX_RX3)
- net RX4+: now also C126.1; no longer MXM1.115 (PEX_RX4#)
- net RX4-: now also C125.1; no longer MXM1.117 (PEX_RX4)
- net RX5+: now also C130.1; no longer MXM1.109 (PEX_RX5#)
- net RX5-: now also C129.1; no longer MXM1.111 (PEX_RX5)
- net RX6+: now also C128.1; no longer MXM1.103 (PEX_RX6#)
- net RX6-: now also C127.1; no longer MXM1.105 (PEX_RX6)
- net RX7+: now also C132.1; no longer MXM1.97 (PEX_RX7#)
- net RX7-: now also C131.1; no longer MXM1.99 (PEX_RX7)
- net RX8+: now also C134.1; no longer MXM1.91 (PEX_RX8#)
- net RX8-: now also C133.1; no longer MXM1.93 (PEX_RX8)
- net RX9+: now also C136.1; no longer MXM1.85 (PEX_RX9#)
- net RX9-: now also C135.1; no longer MXM1.87 (PEX_RX9)
- new net C_RX0+: C118.2, MXM1.147 (PEX_RX0#)
- new net C_RX0-: C117.2, MXM1.149 (PEX_RX0)
- new net C_RX1+: C120.2, MXM1.141 (PEX_RX1#)
- new net C_RX1-: C119.2, MXM1.143 (PEX_RX1)
- new net C_RX10+: C138.2, MXM1.79 (PEX_RX10#)
- new net C_RX10-: C137.2, MXM1.81 (PEX_RX10)
- new net C_RX11+: C140.2, MXM1.73 (PEX_RX11#)
- new net C_RX11-: C139.2, MXM1.75 (PEX_RX11)
- new net C_RX12+: C142.2, MXM1.67 (PEX_RX12#)
- new net C_RX12-: C141.2, MXM1.69 (PEX_RX12)
- new net C_RX13+: C144.2, MXM1.61 (PEX_RX13#)
- new net C_RX13-: C143.2, MXM1.63 (PEX_RX13)
- new net C_RX14+: C146.2, MXM1.55 (PEX_RX14#)
- new net C_RX14-: C145.2, MXM1.57 (PEX_RX14)
- new net C_RX15+: C148.2, MXM1.49 (PEX_RX15#)
- new net C_RX15-: C147.2, MXM1.51 (PEX_RX15)
- new net C_RX2+: C122.2, MXM1.135 (PEX_RX2#)
- new net C_RX2-: C121.2, MXM1.137 (PEX_RX2)
- new net C_RX3+: C124.2, MXM1.121 (PEX_RX3#)
- new net C_RX3-: C123.2, MXM1.123 (PEX_RX3)
- new net C_RX4+: C126.2, MXM1.115 (PEX_RX4#)
- new net C_RX4-: C125.2, MXM1.117 (PEX_RX4)
- new net C_RX5+: C130.2, MXM1.109 (PEX_RX5#)
- new net C_RX5-: C129.2, MXM1.111 (PEX_RX5)
- new net C_RX6+: C128.2, MXM1.103 (PEX_RX6#)
- new net C_RX6-: C127.2, MXM1.105 (PEX_RX6)
- new net C_RX7+: C132.2, MXM1.97 (PEX_RX7#)
- new net C_RX7-: C131.2, MXM1.99 (PEX_RX7)
- new net C_RX8+: C134.2, MXM1.91 (PEX_RX8#)
- new net C_RX8-: C133.2, MXM1.93 (PEX_RX8)
- new net C_RX9+: C136.2, MXM1.85 (PEX_RX9#)
- new net C_RX9-: C135.2, MXM1.87 (PEX_RX9)
Other:
- moved on the sheet: C50, C51, C52, C53, C58, C59, Q17, Q18, Q19, Q20, TP10, TP11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
